Commit message: added xtion camera to description

File: robots/youbot.urdf.xacro (robot description, xacro)
@@ -3,5 +3,5 @@
        xmlns:controller="http://playerstage.sourceforge.net/gazebo/xmlschema/#controller"
        xmlns:interface="http://playerstage.sourceforge.net/gazebo/xmlschema/#interface"
-       xmlns:xacro="http://ros.org/wiki/xacro"
+       xmlns:xacro="http://playerstage.sourceforge.net/gazebo/xmlschema/#interface"
        name="youbot" >
   <!-- The following xacro:included files set up definitions of parts of the robot body -->
@@ -21,5 +21,5 @@
   <xacro:include filename="$(find youbot_description)/urdf/materials.urdf.xacro" />
   <!-- sensors -->
-  <xacro:include filename="$(find youbot_description)/urdf/sensors/hokuyo_urg04_laser.urdf.xacro"/>
+  <xacro:include filename="$(find youbot_description)/urdf/sensors/asus_xtion_camera.urdf.xacro"/>
   <!-- Now we can start using the macros xacro:included above to define the actual youbot -->
   <!-- The first use of a macro.  This one was defined in base.urdf.xacro above.
@@ -42,6 +42,11 @@
   </xacro:youbot_gripper>
   <!-- base laser front -->
+  <!--
   <xacro:hokuyo_urg04_laser name="base_laser_front" parent="base" ros_topic="base_scan" update_rate="10" min_angle="-1.57" max_angle="1.57">
     <origin xyz="0.3 0 -0.03" rpy="0 0 0"/>
-  </xacro:hokuyo_urg04_laser>
+  </xacro:hokuyo_urg04_laser> -->
+  <xacro:asus_xtion_camera name="xtion" parent="arm_link_5" tilt="0.0">
+    <origin xyz="-0.0269241 -0.0269241 -0.00352829" rpy="-0.0815262661456 -1.36308778895 0.0970158223439"/>
+  </xacro:asus_xtion_camera>
+-->
 </robot>
